File: Hardware/Locket.sch (KiCad schematic (older format))
At the start: 76 parts, among them M1 MOTOR_PAD, Q1 LED_RGB 5050, Q2 IRLML9303, Q3 IRLML9303, SW1 SWITCH, SW2 BUTTON, SW3 DIPx4, SW4 SWITCH

Commit message: + Locket hardware v2 * switch to 10 kBit
Parts:
- removed Q2, Q3: IRLML9303, SOT:SOT23-3, symbol IRLML6302
- removed R7: 20k, Resistors:RES_0603, symbol R
- added Q2, Q3: MMBT2222, SOT:SOT23-3, symbol NPN
- added R12, R13: 1k, Resistors:RES_0603, symbol R
- C20, C21: value 10u -> 0.1u; footprint Capacitors:CAP_0805 -> Capacitors:CAP_0603
- DD1: value STM32L151CXTX -> STM32L151CxTx
Connections:
- net LED_EN is gone; now on net ACC_INT1: DD1.40 (PB4/JTRST/T3C1/MISO1)
- net +3.3V: now also BZ1.1, C21.1, DA1.1 (CE), L2.2, L3.2, SW2.2; no longer R4.1, R5.1, R6.1
- net +BATT: now also C22.1, C8.1, D2.C, L1.2, M1.1 (+), XL6.1 (P1); no longer C1.1, C14.1, C15.1, C16.1, C17.1, C18.1, C19.1, C2.1, C3.1, C4.1, C5.1, C6.1, C7.1, C9.1, DD1.1 (VDD), DD1.24 (VDD1), DD1.36 (VDD2), DD1.48 (VDD3), DD1.9 (VDDA), DD2.11 (AVDD), DD2.14 (AVDD), DD2.15 (AVDD), DD2.18 (DGUARD), DD2.4 (DVDD), DD2.9 (AVDD), DD3.1 (VDDIO), DD3.14 (VDD), L2.2, R10.1, R11.2, SW2.2, XL3.1 (Vdd)
- net ACC_INT1: no longer DD1.25 (PB12/CK3/T10C1/ADC18)
- net BLUE_LED: now also R6.1; no longer Q1.BC (B)
- net Buzzer: now also DD1.46 (PB9/SDA1/T4C4/T11C1), R12.1; no longer DD1.39 (PB3/JTDO/T2C2/SCK1)
- net BuzzerOut: now also Q2.3 (C)
- net DS1: now also SW3.8; no longer SW3.1
- net DS2: now also SW3.7; no longer SW3.2
- net DS3: now also SW3.6; no longer SW3.3
- net DS4: now also SW3.5; no longer SW3.4
- net GND: now also C10.2, C21.2, C22.2, C8.2, DA1.4 (GND), M1.PAD (GND), Q1.BC (B), Q1.GC (G), Q1.RC, SW3.1, SW3.2, SW3.3, SW3.4, Q2.2 (E), Q3.2 (E); no longer L3.2, SW3.5, SW3.6, SW3.7, SW3.8
- net GREEN_LED: now also R5.1; no longer Q1.GC (G)
- net PeriphPwr: now also DD1.39 (PB3/JTDO/T2C2/SCK1); no longer DD1.46 (PB9/SDA1/T4C4/T11C1)
- net RED_LED: now also R4.1; no longer Q1.RC
- net Vibro: now also R13.1
- net VibroOut: now also D2.A, XL6.2 (PM), Q3.3 (C); no longer D2.C, XL6.1 (P1)
- removed net GNDPWR: BZ1.1, C10.2, C21.2, C22.2, C8.2, D2.A, DA1.4 (GND), L3.1, M1.1 (+), M1.PAD (GND), XL6.2 (PM)
- removed net PWR_F: C21.1, C22.1, C8.1, L1.2, L2.1
- new net: Q3.1 (B), R13.2
- new net: Q2.1 (B), R12.2
- new net PWR_CC: C14.1, C15.1, C16.1, C17.1, C18.1, C19.1, DD2.11 (AVDD), DD2.14 (AVDD), DD2.15 (AVDD), DD2.18 (DGUARD), DD2.4 (DVDD), DD2.9 (AVDD), L3.1
- new net PWR_MCU: C1.1, C2.1, C3.1, C4.1, C5.1, C6.1, C7.1, C9.1, DD1.1 (VDD), DD1.24 (VDD1), DD1.36 (VDD2), DD1.48 (VDD3), DD1.9 (VDDA), DD3.1 (VDDIO), DD3.14 (VDD), L2.1, R10.1, R11.2, XL3.1 (Vdd)
- no-connect marks 10 -> 11
Other:
- note added: "CC Power Filter"
- note added: "CPU: \nL100, L15x, F030C8, F051C8,\nF100C4(acc sw i2c only), \n"
- note added: "For Locket case:\nC23, C25 - Do Not Mount\nL4 = 5.6nH"
- note added: "MCU Power Filter"
- note added: "Pins 15, 14, 11, 9, 4, 18"
- note added: "Pins 24, 36, 48, 1+9"
- note added: "Power +3V3"
- note removed: "CPU"
- note removed: "Power Filter"
- note removed: "Power for LED"
- moved on the sheet: ANT1, BLN1, BZ1, C1, C10, C14, C15, C16, C17, C18, C19, C2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

Commit message: + Antenna matched, sch updated + Vibro works
Parts:
- C23: value DoNotMount -> 1.5pF
- C25: value 1.5pF -> DoNotMount
- L4: value 33nH -> 5.6nH
Other:
- note added: "PLA Locket case:\nC23 = 1.5pF, \nC25 - Do Not Mount\nL4 = 5.6nH"
- note removed: "For Locket case:\nC23, C25 - Do Not Mount\nL4 = 5.6nH"
Changed lines of the file:
@@
 P 12850 2350
 F 0 "C23" H 12900 2450 50  0000 L CNN
-F 1 "DoNotMount" H 12900 2250 50  0000 L CNN
+F 1 "1.5pF" H 12900 2250 50  0000 L CNN
 F 2 "Capacitors:CAP_0402" H 12850 2350 60  0001 C CNN
 F 3 "" H 12850 2350 60  0001 C CNN
@@
 P 13200 1850
 F 0 "L4" V 13100 1710 40  0000 C CNN
-F 1 "33nH" V 13100 1850 40  0000 C CNN
+F 1 "5.6nH" V 13100 1850 40  0000 C CNN
 F 2 "Inductors:IND_0402" V 13260 1860 40  0000 C CNN
 F 3 "~" H 13200 1850 60  0000 C CNN
@@
 P 13550 2350
 F 0 "C25" H 13600 2450 50  0000 L CNN
-F 1 "1.5pF" H 13600 2250 50  0000 L CNN
+F 1 "DoNotMount" H 13600 2250 50  0000 L CNN
 F 2 "Capacitors:CAP_0402" H 13550 2350 60  0001 C CNN
 F 3 "" H 13550 2350 60  0001 C CNN
@@
 Text Label 13600 1850 0    60   ~ 0
 ANT2
-Text Notes 12850 2900 0    60   ~ 0
-For Locket case:\nC23, C25 - Do Not Mount\nL4 = 5.6nH
 $Comp
 L NPN Q3
@@
 Text Label 2000 5750 0    60   ~ 0
 PWR_MCU
+Text Notes 12850 3000 0    60   ~ 0
+PLA Locket case:\nC23 = 1.5pF, \nC25 - Do Not Mount\nL4 = 5.6nH
 $EndSCHEMATC

Commit message: Proceeding
Parts:
- removed DD3: MMA8452Q, QFN:QFN16_5_3, symbol MMA8452Q
- removed M1: MOTOR_PAD, Installations:MOTOR_KHN4NX, symbol MOTOR_PAD
- removed SW1: SWITCH, Switches:SW_SS-6, symbol SWITCH
- removed XL2: CONN_2, Connectors:PLS-2, symbol CONN_2
- added C?: 1000u 6v3, symbol CP
- C1: value 10u -> 4.7u; footprint Capacitors:CAP_0805 -> Capacitors:CAP_0603
Connections:
- net labels added: PwrMCU, VCC
- net labels removed: PWR_CC
- wire segments 241 -> 237
- no-connect marks 11 -> 9
Other:
- note added: "Keep CS High\nwhen sleep"
- note removed: "Battery 3V"
- note removed: "Choose one of two footprints"
- note removed: "Choose one or another motor"
- moved on the sheet: B1, B2, C24, C7, C9, D2, Q1, R4, R5, R6, R9, SW2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

Commit message: + 9D mems
Parts:
- removed C21, C24: 0.1u, Capacitors:CAP_0603, symbol C
- removed L3: TB201209 G152, Inductors:IND_0805, symbol L
- removed XL5: CONN_4, Connectors:PLS-4, symbol CONN_4
- added C?: 0.1u, symbol C
- added C?: 4.7u, CAP_0603, symbol C
- added C?: 0.22u, CAP_0603, symbol C
- added DD?: LSM9DS0, symbol LSM9DS0
- added L?: BLM15AG102SN1, Inductors:IND_0402, symbol L
- added Q?: TSOP75256, symbol TSOP752XX
- added R?: 100, symbol R
- L2: value TB201209 G152 -> BLM15AG102SN1; footprint Inductors:IND_0805 -> Inductors:IND_0402
Connections:
- net labels added: GYRO_DRDY, IR_In, IR_Power, LED_EN
- net labels removed: PWR_MCU
- wire segments 237 -> 257
Other:
- note added: "Accelerometer/Magnetic: I2C addr = 0011110 (0x1E)\n Gyroscope: I2C addr = 1101010 (0x6A)"
- note added: "Address\nLSB"
- note added: "I2C Bus\nEnabled"
- note added: "Keep away from motor, power lines etc."
- note added: "Periphery\n\nPA0: WKUP\nT3 C2, 3, 4: LED RGB\nT4C4: buzzer\nT10C1: IR_In\nI2C1: Pill \nI2C2: MEMS Sns\nSPI1: CC\nUART1: Debug UART"
- note removed: "Accelerometer\nI2C addr = 0x1C"
- note removed: "Just\nPins"
- moved on the sheet: C10, C20, C7, C8, C9, D1, DA1, L1, RP1, RP2, SW2
